Commit message: support mid360 laserscan

File: aloha_description/arx5_description/urdf/arx5_description.urdf (robot description, URDF)
Before this commit: robot arx5_description, 39 links, 39 joints
Links:
- added link robot::footprint
Joints:
- added joint livox_joint: type fixed, parent footprint, child livox_base, origin xyz=0.23 0 0.19 rpy=0 0 0, axis 0 0 0
- added joint robot_footprint_joint: type fixed, parent footprint, child robot::footprint, origin xyz=0.18 0 0.29 rpy=0 0 0, axis 0 0 0

File: aloha_description/livox_laser_simulation/urdf/livox_mid360.xacro (robot description, xacro)
@@ -17,5 +17,5 @@
   <xacro:macro name="Livox_Mid_gazebo_sensor" params="visualize:=True update_rate:=10 resolution:=0.002 noise_mean:=0.0 noise_stddev:=0.01 name:=livox">
     <gazebo reference="${name}">
-      <sensor type="ray" name="laser_${name}">
+      <sensor type="ray" name="${name}">
         <pose>0 0 0 0 0 0</pose>
         <visualize>${visualize}</visualize>
@@ -62,14 +62,16 @@
       <xacro:null_inertial/>
       <visual>
-        <origin xyz="0.00 0 0.0" rpy="0 0 0"/>
+        <origin xyz="0.00 0 0.0" rpy="1.57 0 3.14"/>
         <geometry>
-          <mesh filename="package://livox_laser_simulation/meshes/livox_mid40.dae">
+          <mesh filename="package://livox_laser_simulation/meshes/livox_mid360.dae" scale="0.001 0.001 0.001">
           </mesh>
         </geometry>
       </visual>
       <collision>
-		  <origin xyz="0 0 0" rpy="0 0 0" /> <geometry> <mesh
-		  filename="package://livox_laser_simulation/meshes/livox_mid40.dae">
-		  </mesh> </geometry>
+		  <origin xyz="0 0 0" rpy="1.57 0 3.14" />
+      <geometry>
+        <mesh filename="package://livox_laser_simulation/meshes/livox_mid360.dae" scale="0.001 0.001 0.001">
+        </mesh>
+      </geometry>
       </collision>
     </link>
@@ -78,12 +80,13 @@
     </link>
     <joint name="${name}_to_${name}_base_joint" type="fixed">
+      <origin rpy="0 0 0" xyz="0.0 0.0 0.03"/>
       <parent link="${name}_base"/>
       <child link="${name}"/>
-      <origin rpy="0 0 0" xyz="0.0 1.0 0.2"/>
+      <axis xyz="0 0 0" />
     </joint>
     <xacro:Livox_Mid_gazebo_sensor name="${name}" visualize="${visualize}"/>
   </xacro:macro>
     <xacro:Livox_Mid40 name="livox"/>
-  <xacro:include filename="$(find livox_laser_simulation)/urdf/standardrobots_oasis300.xacro"/>
-  <xacro:link_oasis name="oasis"/>
+  <!-- <xacro:include filename="$(find livox_laser_simulation)/urdf/standardrobots_oasis300.xacro"/>
+  <xacro:link_oasis name="oasis"/> -->
 </robot>
