Commit message: 修改机械臂零点

File: aloha_new_description/urdf/aloha_new_v00.urdf (robot description, URDF)
Before this commit: robot arx5_description, 50 links, 49 joints
Joints:
- joint bl_joint2: origin xyz=0 0 0 rpy=1.5708 -0.10095 -1.5708 -> xyz=0 0 0 rpy=1.5708 -0.135857 -1.5708
- joint bl_joint3: origin xyz=0.28503 0 0 rpy=0 0 1.3826 -> xyz=0.28503 0 0 rpy=0 0 1.347693
- joint br_joint2: origin xyz=0 0 0 rpy=1.5708 -0.10095 -1.5708 -> xyz=0 0 0 rpy=1.5708 -0.135857 -1.5708
- joint br_joint3: origin xyz=0.28503 0 0 rpy=0 0 1.3826 -> xyz=0.28503 0 0 rpy=0 0 1.347693
- joint fl_joint2: origin xyz=0 0 0 rpy=1.5708 -0.10095 -1.5708 -> xyz=0 0 0 rpy=1.5708 -0.135857 -1.5708
- joint fl_joint3: origin xyz=0.28503 0 0 rpy=0 0 1.3826 -> xyz=0.28503 0 0 rpy=0 0 1.347693
- joint fr_joint2: origin xyz=0 0 0 rpy=1.5708 -0.10095 -1.5708 -> xyz=0 0 0 rpy=1.5708 -0.135857 -1.5708
- joint fr_joint3: origin xyz=0.28503 0 0 rpy=0 0 1.3826 -> xyz=0.28503 0 0 rpy=0 0 1.347693
