Commit message: 增加渲染

File: aloha_new_description/urdf/aloha_new.urdf (robot description, URDF)
Before this commit: robot arx5_description, 50 links, 49 joints
Links:
- link bl_base_link: geometry collision mesh filename=package://aloha_new_description/meshes/base_link.STL; visual mesh filename=package://aloha_new_description/meshes/base_link.dae
- link bl_link1: geometry collision mesh filename=package://aloha_new_description/meshes/link1.STL; visual mesh filename=package://aloha_new_description/meshes/link1.dae
- link bl_link2: geometry collision mesh filename=package://aloha_new_description/meshes/link2.STL; visual mesh filename=package://aloha_new_description/meshes/link2.dae
- link bl_link3: geometry collision mesh filename=package://aloha_new_description/meshes/link3.STL; visual mesh filename=package://aloha_new_description/meshes/link3.dae
- link bl_link4: geometry collision mesh filename=package://aloha_new_description/meshes/link4.STL; visual mesh filename=package://aloha_new_description/meshes/link4.dae
- link bl_link5: geometry collision mesh filename=package://aloha_new_description/meshes/link5.STL; visual mesh filename=package://aloha_new_description/meshes/link5.dae
- link body_Link: geometry collision mesh filename=package://aloha_new_description/meshes/body.dae; visual mesh filename=package://aloha_new_description/meshes/body.dae
- link br_base_link: geometry collision mesh filename=package://aloha_new_description/meshes/base_link.STL; visual mesh filename=package://aloha_new_description/meshes/base_link.dae
- link br_link1: geometry collision mesh filename=package://aloha_new_description/meshes/link1.STL; visual mesh filename=package://aloha_new_description/meshes/link1.dae
- link br_link2: geometry collision mesh filename=package://aloha_new_description/meshes/link2.STL; visual mesh filename=package://aloha_new_description/meshes/link2.dae
- link br_link3: geometry collision mesh filename=package://aloha_new_description/meshes/link3.STL; visual mesh filename=package://aloha_new_description/meshes/link3.dae
- link br_link4: geometry collision mesh filename=package://aloha_new_description/meshes/link4.STL; visual mesh filename=package://aloha_new_description/meshes/link4.dae
- link br_link5: geometry collision mesh filename=package://aloha_new_description/meshes/link5.STL; visual mesh filename=package://aloha_new_description/meshes/link5.dae
- link fl_base_link: geometry collision mesh filename=package://aloha_new_description/meshes/base_link.STL; visual mesh filename=package://aloha_new_description/meshes/base_link.dae
- link fl_link1: geometry collision mesh filename=package://aloha_new_description/meshes/link1.STL; visual mesh filename=package://aloha_new_description/meshes/link1.dae
- link fl_link2: geometry collision mesh filename=package://aloha_new_description/meshes/link2.STL; visual mesh filename=package://aloha_new_description/meshes/link2.dae
- link fl_link3: geometry collision mesh filename=package://aloha_new_description/meshes/link3.STL; visual mesh filename=package://aloha_new_description/meshes/link3.dae
- link fl_link4: geometry collision mesh filename=package://aloha_new_description/meshes/link4.STL; visual mesh filename=package://aloha_new_description/meshes/link4.dae
- link fl_link5: geometry collision mesh filename=package://aloha_new_description/meshes/link5.STL; visual mesh filename=package://aloha_new_description/meshes/link5.dae
- link fr_base_link: geometry collision mesh filename=package://aloha_new_description/meshes/base_link.STL; visual mesh filename=package://aloha_new_description/meshes/base_link.dae
- link fr_link1: geometry collision mesh filename=package://aloha_new_description/meshes/link1.STL; visual mesh filename=package://aloha_new_description/meshes/link1.dae
- link fr_link2: geometry collision mesh filename=package://aloha_new_description/meshes/link2.STL; visual mesh filename=package://aloha_new_description/meshes/link2.dae
- link fr_link3: geometry collision mesh filename=package://aloha_new_description/meshes/link3.STL; visual mesh filename=package://aloha_new_description/meshes/link3.dae
- link fr_link4: geometry collision mesh filename=package://aloha_new_description/meshes/link4.STL; visual mesh filename=package://aloha_new_description/meshes/link4.dae
- link fr_link5: geometry collision mesh filename=package://aloha_new_description/meshes/link5.STL; visual mesh filename=package://aloha_new_description/meshes/link5.dae
Joints:
- removed joint body
- added joint base_joint: type fixed, parent footprint, child base_link, origin xyz=0 0 0.15 rpy=0 0 0, axis 0 0 0
- joint body_joint: child base_link -> body_Link; origin xyz=0 0 0.15 rpy=0 0 0 -> xyz=0 0 0 rpy=0 0 0
- joint fl_joint2: origin xyz=0 0 0 rpy=1.5708 -0.18822 -1.5708 -> xyz=0 0 0 rpy=1.5708 -0.10095 -1.5708

Commit message: 修改urdf颜色,令其显眼

File: aloha_new_description/urdf/aloha_new.urdf (robot description, URDF)
Before this commit: robot arx5_description, 50 links, 49 joints
Links:
- link bl_base_link: mass 0.162352169522719 -> 0.162548567403693
- link bl_link1: mass 0.0978679932242824 -> 0.0978679932242826
- link bl_link2: mass 0.289570182962832 -> 0.290888938633388
- link bl_link3: mass 0.29058359696822 -> 0.290847805579065
- link bl_link4: mass 0.12708738799602 -> 0.127087348341362
- link bl_link5: mass 0.144711209371805 -> 0.144711242639457
- link bl_link6: mass 0.214619655313844 -> 0.214619908036656; geometry collision mesh filename=package://aloha_new_description/meshes/piper_slave_meshes/l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; visual mesh filename=package://aloha_new_description/meshes/piper_slave_meshes/l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
- link bl_link7: mass 0.0163980778203027 -> 0.0163980774922961; geometry collision mesh filename=package://aloha_new_description/meshes/piper_slave_meshes/l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; visual mesh filename=package://aloha_new_description/meshes/piper_slave_meshes/l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
- link bl_link8: mass 0.0159830776295144 -> 0.0159830768118613; geometry collision mesh filename=package://aloha_new_description/meshes/piper_slave_meshes/l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; visual mesh filename=package://aloha_new_description/meshes/piper_slave_meshes/l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
- link br_base_link: mass 0.162352169522719 -> 0.162548567403693
- link br_link1: mass 0.0978679932242824 -> 0.0978679932242826
- link br_link2: mass 0.289570182962832 -> 0.290888938633388
- link br_link3: mass 0.29058359696822 -> 0.290847805579065
- link br_link4: mass 0.12708738799602 -> 0.127087348341362
- link br_link5: mass 0.144711209371805 -> 0.144711242639457
- link br_link6: mass 0.214619655313844 -> 0.214619908036656; geometry collision mesh filename=package://aloha_new_description/meshes/piper_slave_meshes/l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; visual mesh filename=package://aloha_new_description/meshes/piper_slave_meshes/l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
- link br_link7: mass 0.0163980778203027 -> 0.0163980774922961; geometry collision mesh filename=package://aloha_new_description/meshes/piper_slave_meshes/l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; visual mesh filename=package://aloha_new_description/meshes/piper_slave_meshes/l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
- link br_link8: mass 0.0159830776295144 -> 0.0159830768118613; geometry collision mesh filename=package://aloha_new_description/meshes/piper_slave_meshes/l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; visual mesh filename=package://aloha_new_description/meshes/piper_slave_meshes/l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
- link fl_base_link: mass 0.162352169522719 -> 0.162548567403693
- link fl_link1: mass 0.0978679932242826 -> 0.0978679932242825
- link fl_link2: mass 0.289570165726093 -> 0.290888938633388
- link fl_link3: mass 0.290583612813414 -> 0.290847697793211
- link fl_link4: mass 0.12708738799602 -> 0.127087348341362
- link fl_link5: mass 0.144711209371806 -> 0.144711242639457
- link fl_link6: mass 0.195186215018024 -> 0.195187143240719
- link fl_link7: mass 0.0264822468303309 -> 0.02648229234527
- link fl_link8: mass 0.0264822458559721 -> 0.0264822021416248
- link fr_base_link: mass 0.162352169522719 -> 0.162548567403693
- link fr_link1: mass 0.0978679932242826 -> 0.0978679932242825
- link fr_link2: mass 0.289570165726093 -> 0.290888938633388
- link fr_link3: mass 0.290583612813414 -> 0.290847697793211
- link fr_link4: mass 0.12708738799602 -> 0.127087348341362
- link fr_link5: mass 0.144711209371806 -> 0.144711242639457
- link fr_link6: mass 0.195186215018024 -> 0.195187143240719
- link fr_link7: mass 0.0264822468303309 -> 0.02648229234527
- link fr_link8: mass 0.0264822458559721 -> 0.0264822021416248
Joints:
- joint bl_joint2: origin xyz=0 0 0 rpy=1.5708 -0.10095 -1.5708 -> xyz=0 0 0 rpy=1.5708 0 -1.5708
- joint bl_joint3: origin xyz=0.28503 0 0 rpy=0 0 1.3826 -> xyz=0.28358 0.028726 0 rpy=0 0 0.10095
- joint bl_joint4: axis 0 0 -1 -> 0 0 1; origin xyz=0.021984 0.25075 0 rpy=-1.5708 0 0 -> xyz=-0.24221 0.068514 0 rpy=-1.5708 0 1.3826
- joint bl_joint6: axis 0 0 -1 -> 0 0 1
- joint bl_joint7: limit lower=0 upper=0.036 effort=10 velocity=1 -> lower=0 upper=0.04 effort=10 velocity=1
- joint bl_joint8: limit lower=-0.036 upper=0 effort=10 velocity=1 -> lower=-0.04 upper=0 effort=10 velocity=1
- joint br_joint2: origin xyz=0 0 0 rpy=1.5708 -0.10095 -1.5708 -> xyz=0 0 0 rpy=1.5708 0 -1.5708
- joint br_joint3: origin xyz=0.28503 0 0 rpy=0 0 1.3826 -> xyz=0.28358 0.028726 0 rpy=0 0 0.10095
- joint br_joint4: axis 0 0 -1 -> 0 0 1; origin xyz=0.021984 0.25075 0 rpy=-1.5708 0 0 -> xyz=-0.24221 0.068514 0 rpy=-1.5708 0 1.3826
- joint br_joint6: axis 0 0 -1 -> 0 0 1
- joint br_joint7: limit lower=0 upper=0.036 effort=10 velocity=1 -> lower=0 upper=0.04 effort=10 velocity=1
- joint br_joint8: limit lower=-0.036 upper=0 effort=10 velocity=1 -> lower=-0.04 upper=0 effort=10 velocity=1
- joint fl_joint2: origin xyz=0 0 0 rpy=1.5708 -0.10095 -1.5708 -> xyz=0 0 0 rpy=1.5708 0 -1.5708
- joint fl_joint3: origin xyz=0.28503 0 0 rpy=0 0 1.3826 -> xyz=0.28358 0.028726 0 rpy=0 0 0.10095
- joint fl_joint4: axis 0 0 -1 -> 0 0 1; origin xyz=0.021984 0.25075 0 rpy=-1.5708 0 0 -> xyz=-0.24221 0.068514 0 rpy=-1.5708 0 1.3826
- joint fl_joint6: axis 0 0 -1 -> 0 0 1
- joint fl_joint7: origin xyz=0 0 0.13503 rpy=1.5708 0 1.5898 -> xyz=0 0 0.13503 rpy=1.5708 0 1.5708
- joint fl_joint8: origin xyz=0 0 0.13503 rpy=-1.5708 0 1.5898 -> xyz=0 0 0.13503 rpy=-1.5708 0 1.5708
- joint fr_joint2: origin xyz=0 0 0 rpy=1.5708 -0.10095 -1.5708 -> xyz=0 0 0 rpy=1.5708 0 -1.5708
- joint fr_joint3: origin xyz=0.28503 0 0 rpy=0 0 1.3826 -> xyz=0.28358 0.028726 0 rpy=0 0 0.10095
- joint fr_joint4: axis 0 0 -1 -> 0 0 1; origin xyz=0.021984 0.25075 0 rpy=-1.5708 0 0 -> xyz=-0.24221 0.068514 0 rpy=-1.5708 0 1.3826
- joint fr_joint6: axis 0 0 -1 -> 0 0 1
- joint fr_joint7: origin xyz=0 0 0.13503 rpy=1.5708 0 1.5898 -> xyz=0 0 0.13503 rpy=1.5708 0 1.5708
- joint fr_joint8: origin xyz=0 0 0.13503 rpy=-1.5708 0 1.5898 -> xyz=0 0 0.13503 rpy=-1.5708 0 1.5708

File: aloha_new_description/urdf/aloha_new_v00.urdf (robot description, URDF)
Before this commit: robot arx5_description, 50 links, 49 joints
Links:
- link bl_base_link: mass 0.162352169522719 -> 0.162548567403693
- link bl_link1: mass 0.0978679932242824 -> 0.0978679932242826
- link bl_link2: mass 0.289570182962832 -> 0.290888938633388
- link bl_link3: mass 0.29058359696822 -> 0.290847805579065
- link bl_link4: mass 0.12708738799602 -> 0.127087348341362
- link bl_link5: mass 0.144711209371805 -> 0.144711242639457
- link bl_link6: mass 0.214619655313844 -> 0.214619908036656; geometry collision mesh filename=package://aloha_new_description/meshes/piper_slave_meshes/l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; visual mesh filename=package://aloha_new_description/meshes/piper_slave_meshes/l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
- link bl_link7: mass 0.0163980778203027 -> 0.0163980774922961; geometry collision mesh filename=package://aloha_new_description/meshes/piper_slave_meshes/l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; visual mesh filename=package://aloha_new_description/meshes/piper_slave_meshes/l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
- link bl_link8: mass 0.0159830776295144 -> 0.0159830768118613; geometry collision mesh filename=package://aloha_new_description/meshes/piper_slave_meshes/l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; visual mesh filename=package://aloha_new_description/meshes/piper_slave_meshes/l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
- link br_base_link: mass 0.162352169522719 -> 0.162548567403693
- link br_link1: mass 0.0978679932242824 -> 0.0978679932242826
- link br_link2: mass 0.289570182962832 -> 0.290888938633388
- link br_link3: mass 0.29058359696822 -> 0.290847805579065
- link br_link4: mass 0.12708738799602 -> 0.127087348341362
- link br_link5: mass 0.144711209371805 -> 0.144711242639457
- link br_link6: mass 0.214619655313844 -> 0.214619908036656; geometry collision mesh filename=package://aloha_new_description/meshes/piper_slave_meshes/l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; visual mesh filename=package://aloha_new_description/meshes/piper_slave_meshes/l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
- link br_link7: mass 0.0163980778203027 -> 0.0163980774922961; geometry collision mesh filename=package://aloha_new_description/meshes/piper_slave_meshes/l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; visual mesh filename=package://aloha_new_description/meshes/piper_slave_meshes/l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
- link br_link8: mass 0.0159830776295144 -> 0.0159830768118613; geometry collision mesh filename=package://aloha_new_description/meshes/piper_slave_meshes/l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; visual mesh filename=package://aloha_new_description/meshes/piper_slave_meshes/l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
- link fl_base_link: mass 0.162352169522719 -> 0.162548567403693
- link fl_link1: mass 0.0978679932242826 -> 0.0978679932242825
- link fl_link2: mass 0.289570165726093 -> 0.290888938633388
- link fl_link3: mass 0.290583612813414 -> 0.290847697793211
- link fl_link4: mass 0.12708738799602 -> 0.127087348341362
- link fl_link5: mass 0.144711209371806 -> 0.144711242639457
- link fl_link6: mass 0.195186215018024 -> 0.195187143240719
- link fl_link7: mass 0.0264822468303309 -> 0.02648229234527
- link fl_link8: mass 0.0264822458559721 -> 0.0264822021416248
- link fr_base_link: mass 0.162352169522719 -> 0.162548567403693
- link fr_link1: mass 0.0978679932242826 -> 0.0978679932242825
- link fr_link2: mass 0.289570165726093 -> 0.290888938633388
- link fr_link3: mass 0.290583612813414 -> 0.290847697793211
- link fr_link4: mass 0.12708738799602 -> 0.127087348341362
- link fr_link5: mass 0.144711209371806 -> 0.144711242639457
- link fr_link6: mass 0.195186215018024 -> 0.195187143240719
- link fr_link7: mass 0.0264822468303309 -> 0.02648229234527
- link fr_link8: mass 0.0264822458559721 -> 0.0264822021416248
Joints:
- joint bl_joint2: origin xyz=0 0 0 rpy=1.5708 -0.135857 -1.5708 -> xyz=0 0 0 rpy=1.5708 -0.034907 -1.5708
- joint bl_joint3: origin xyz=0.28503 0 0 rpy=0 0 1.347693 -> xyz=0.28358 0.028726 0 rpy=0 0 0.06604341
- joint bl_joint4: axis 0 0 -1 -> 0 0 1; origin xyz=0.021984 0.25075 0 rpy=-1.5708 0 0 -> xyz=-0.24221 0.068514 0 rpy=-1.5708 0 1.3826
- joint bl_joint6: axis 0 0 -1 -> 0 0 1
- joint bl_joint7: limit lower=0 upper=0.036 effort=10 velocity=1 -> lower=0 upper=0.04 effort=10 velocity=1
- joint bl_joint8: limit lower=-0.036 upper=0 effort=10 velocity=1 -> lower=-0.04 upper=0 effort=10 velocity=1
- joint br_joint2: origin xyz=0 0 0 rpy=1.5708 -0.135857 -1.5708 -> xyz=0 0 0 rpy=1.5708 -0.034907 -1.5708
- joint br_joint3: origin xyz=0.28503 0 0 rpy=0 0 1.347693 -> xyz=0.28358 0.028726 0 rpy=0 0 0.06604341
- joint br_joint4: axis 0 0 -1 -> 0 0 1; origin xyz=0.021984 0.25075 0 rpy=-1.5708 0 0 -> xyz=-0.24221 0.068514 0 rpy=-1.5708 0 1.3826
- joint br_joint6: axis 0 0 -1 -> 0 0 1
- joint br_joint7: limit lower=0 upper=0.036 effort=10 velocity=1 -> lower=0 upper=0.04 effort=10 velocity=1
- joint br_joint8: limit lower=-0.036 upper=0 effort=10 velocity=1 -> lower=-0.04 upper=0 effort=10 velocity=1
- joint fl_joint2: origin xyz=0 0 0 rpy=1.5708 -0.135857 -1.5708 -> xyz=0 0 0 rpy=1.5708 -0.034907 -1.5708
- joint fl_joint3: origin xyz=0.28503 0 0 rpy=0 0 1.347693 -> xyz=0.28358 0.028726 0 rpy=0 0 0.06604341
- joint fl_joint4: axis 0 0 -1 -> 0 0 1; origin xyz=0.021984 0.25075 0 rpy=-1.5708 0 0 -> xyz=-0.24221 0.068514 0 rpy=-1.5708 0 1.3826
- joint fl_joint6: axis 0 0 -1 -> 0 0 1
- joint fl_joint7: origin xyz=0 0 0.13503 rpy=1.5708 0 1.5898 -> xyz=0 0 0.13503 rpy=1.5708 0 1.5708
- joint fl_joint8: origin xyz=0 0 0.13503 rpy=-1.5708 0 1.5898 -> xyz=0 0 0.13503 rpy=-1.5708 0 1.5708
- joint fr_joint2: origin xyz=0 0 0 rpy=1.5708 -0.135857 -1.5708 -> xyz=0 0 0 rpy=1.5708 -0.034907 -1.5708
- joint fr_joint3: origin xyz=0.28503 0 0 rpy=0 0 1.347693 -> xyz=0.28358 0.028726 0 rpy=0 0 0.06604341
- joint fr_joint4: axis 0 0 -1 -> 0 0 1; origin xyz=0.021984 0.25075 0 rpy=-1.5708 0 0 -> xyz=-0.24221 0.068514 0 rpy=-1.5708 0 1.3826
- joint fr_joint6: axis 0 0 -1 -> 0 0 1
- joint fr_joint7: origin xyz=0 0 0.13503 rpy=1.5708 0 1.5898 -> xyz=0 0 0.13503 rpy=1.5708 0 1.5708
- joint fr_joint8: origin xyz=0 0 0.13503 rpy=-1.5708 0 1.5898 -> xyz=0 0 0.13503 rpy=-1.5708 0 1.5708

Commit message: Update aloha_new.urdf
修正主臂的模型使用的是从臂模型的问题

File: aloha_new_description/urdf/aloha_new.urdf (robot description, URDF)
Before this commit: robot arx5_description, 50 links, 49 joints
Links:
- link bl_link6: geometry collision mesh filename=package://aloha_new_description/meshes/piper_master_meshes/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; visual mesh filename=package://aloha_new_description/meshes/piper_master_meshes/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
- link bl_link7: geometry collision mesh filename=package://aloha_new_description/meshes/piper_master_meshes/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; visual mesh filename=package://aloha_new_description/meshes/piper_master_meshes/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
- link bl_link8: geometry collision mesh filename=package://aloha_new_description/meshes/piper_master_meshes/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; visual mesh filename=package://aloha_new_description/meshes/piper_master_meshes/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
- link br_link6: geometry collision mesh filename=package://aloha_new_description/meshes/piper_master_meshes/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; visual mesh filename=package://aloha_new_description/meshes/piper_master_meshes/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
- link br_link7: geometry collision mesh filename=package://aloha_new_description/meshes/piper_master_meshes/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; visual mesh filename=package://aloha_new_description/meshes/piper_master_meshes/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
- link br_link8: geometry collision mesh filename=package://aloha_new_description/meshes/piper_master_meshes/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; visual mesh filename=package://aloha_new_description/meshes/piper_master_meshes/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
