Commit message: 增加多个aloha定制版本

File: aloha_new_description/urdf/aloha_tracer2.urdf (robot description, URDF)
Before this commit: robot aloha_description, 45 links, 44 joints
Links:
- added link camera_stand_1_Link, mass 3.736; collision mesh filename=package://aloha_new_description/meshes/camera_stand_1.dae; visual mesh filename=package://aloha_new_description/meshes/camera_stand_1.dae
- added link camera_stand_2_Link, mass 3.736; collision mesh filename=package://aloha_new_description/meshes/camera_stand_2.dae; visual mesh filename=package://aloha_new_description/meshes/camera_stand_2.dae
- link body_Link: geometry collision mesh filename=package://aloha_new_description/meshes/body_v2.dae; visual mesh filename=package://aloha_new_description/meshes/body_v2.dae
Joints:
- added joint camera_stand_1_joint: type prismatic, parent body_Link, child camera_stand_1_Link, origin xyz=0.18 0 0.87 rpy=0 0 0, axis 0 0 1, limit lower=0 upper=0.5 effort=10 velocity=1
- added joint camera_stand_2_joint: type revolute, parent camera_stand_1_Link, child camera_stand_2_Link, origin xyz=0.043 0.0 -0.002 rpy=0 0 0, axis 0 1 0, limit lower=-0.52 upper=0.52 effort=10 velocity=1.0
- added joint d435_camera_joint: type fixed, parent camera_stand_2_Link, child d435_camera_link, origin xyz=0.0 0.0 0.0 rpy=0.0 0.0 0.0, axis 0.0 0.0 0.0, limit lower=0.0 upper=0.0 effort=0.0 velocity=0.0
