Commit message: add tracer2.dae

File: aloha_new_description/urdf/aloha_tracer2_d435.urdf (robot description, URDF)
Before this commit: robot aloha_description, 58 links, 57 joints
Links:
- link base_link: geometry collision mesh filename=package://tracer2_description/meshes/base_link.STL; visual mesh filename=package://aloha_new_description/meshes/tracer2.dae
- link camera_link: geometry collision mesh filename=package://realsense2_description/meshes/d435.dae; visual mesh filename=package://realsense2_description/meshes/d435.dae
- link fl_camera_link: geometry collision mesh filename=package://realsense2_description/meshes/d435.dae; visual mesh filename=package://realsense2_description/meshes/d435.dae
- link fr_camera_link: geometry collision mesh filename=package://realsense2_description/meshes/d435.dae; visual mesh filename=package://realsense2_description/meshes/d435.dae

File: aloha_new_description/urdf/aloha_tracer2_d435_dark.urdf (robot description, URDF)
Before this commit: robot aloha_description, 58 links, 57 joints
Links:
- link base_link: geometry collision mesh filename=package://tracer2_description/meshes/base_link.STL; visual mesh filename=package://aloha_new_description/meshes/tracer2.dae
- link camera_link: geometry collision mesh filename=package://realsense2_description/meshes/d435.dae; visual mesh filename=package://realsense2_description/meshes/d435.dae
- link fl_camera_link: geometry collision mesh filename=package://realsense2_description/meshes/d435.dae; visual mesh filename=package://realsense2_description/meshes/d435.dae
- link fr_camera_link: geometry collision mesh filename=package://realsense2_description/meshes/d435.dae; visual mesh filename=package://realsense2_description/meshes/d435.dae

File: aloha_new_description/urdf/aloha_tracer2_dabai_dark.urdf (robot description, URDF)
Before this commit: robot aloha_description, 52 links, 51 joints
Links:
- link base_link: geometry collision mesh filename=package://tracer2_description/meshes/base_link.STL; visual mesh filename=package://aloha_new_description/meshes/tracer2.dae

File: aloha_new_description/urdf/aloha_tracer2_four_d435_dark.urdf (robot description, URDF)
Before this commit: robot aloha_description, 60 links, 59 joints
Links:
- link base_link: geometry collision mesh filename=package://tracer2_description/meshes/base_link.STL; visual mesh filename=package://aloha_new_description/meshes/tracer2.dae
- link fl_camera_link: geometry collision mesh filename=package://realsense2_description/meshes/d435.dae; visual mesh filename=package://realsense2_description/meshes/d435.dae
- link fr_camera_link: geometry collision mesh filename=package://realsense2_description/meshes/d435.dae; visual mesh filename=package://realsense2_description/meshes/d435.dae
