Commit message: 统一collision和visual

File: aloha_new_description/urdf/aloha_tracer2_d435_dark.urdf (robot description, URDF)
Before this commit: robot aloha_description, 58 links, 57 joints
Links:
- link bl_base_link: geometry collision mesh filename=package://aloha_new_description/meshes/dark_dae/base_link.d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; visual mesh filename=package://aloha_new_description/meshes/dark_dae/base_link.d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
- link bl_link5: geometry collision mesh filename=package://aloha_new_description/meshes/dark_dae/link5.dae; visual mesh filename=package://aloha_new_description/meshes/dark_dae/link5.dae
- link bl_link6: geometry collision mesh filename=package://aloha_new_description/meshes/dark_dae/link6_.dae; visual mesh filename=package://aloha_new_description/meshes/dark_dae/link6_.dae
- link bl_link7: geometry collision mesh filename=package://aloha_new_description/meshes/dark_dae/link7_maste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; visual mesh filename=package://aloha_new_description/meshes/dark_dae/link7_maste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
- link bl_link8: geometry collision mesh filename=package://aloha_new_description/meshes/dark_dae/link8_maste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; visual mesh filename=package://aloha_new_description/meshes/dark_dae/link8_maste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
- link br_base_link: geometry collision mesh filename=package://aloha_new_description/meshes/dark_dae/base_link.d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; visual mesh filename=package://aloha_new_description/meshes/dark_dae/base_link.d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
- link br_link5: geometry collision mesh filename=package://aloha_new_description/meshes/dark_dae/link5.dae; visual mesh filename=package://aloha_new_description/meshes/dark_dae/link5.dae
- link br_link6: geometry collision mesh filename=package://aloha_new_description/meshes/dark_dae/link6_.dae; visual mesh filename=package://aloha_new_description/meshes/dark_dae/link6_.dae
- link br_link7: geometry collision mesh filename=package://aloha_new_description/meshes/dark_dae/link7_maste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; visual mesh filename=package://aloha_new_description/meshes/dark_dae/link7_maste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
- link br_link8: geometry collision mesh filename=package://aloha_new_description/meshes/dark_dae/link8_maste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; visual mesh filename=package://aloha_new_description/meshes/dark_dae/link8_maste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
- link fl_base_link: geometry collision mesh filename=package://aloha_new_description/meshes/dark_dae/base_link.d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; visual mesh filename=package://aloha_new_description/meshes/dark_dae/base_link.d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
- link fl_link5: geometry collision mesh filename=package://aloha_new_description/meshes/dark_dae/link5.dae; visual mesh filename=package://aloha_new_description/meshes/dark_dae/link5.dae
- link fr_base_link: geometry collision mesh filename=package://aloha_new_description/meshes/dark_dae/base_link.d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; visual mesh filename=package://aloha_new_description/meshes/dark_dae/base_link.d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
- link fr_link5: geometry collision mesh filename=package://aloha_new_description/meshes/dark_dae/link5.dae; visual mesh filename=package://aloha_new_description/meshes/dark_dae/link5.dae

File: aloha_new_description/urdf/aloha_tracer2_dabai_dark.urdf (robot description, URDF)
Before this commit: robot aloha_description, 52 links, 51 joints
Links:
- link bl_base_link: geometry collision mesh filename=package://aloha_new_description/meshes/dark_dae/base_link.d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; visual mesh filename=package://aloha_new_description/meshes/dark_dae/base_link.d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
- link bl_link5: geometry collision mesh filename=package://aloha_new_description/meshes/dark_dae/link5.dae; visual mesh filename=package://aloha_new_description/meshes/dark_dae/link5.dae
- link bl_link6: geometry collision mesh filename=package://aloha_new_description/meshes/dark_dae/link6_.dae; visual mesh filename=package://aloha_new_description/meshes/dark_dae/link6_.dae
- link bl_link7: geometry collision mesh filename=package://aloha_new_description/meshes/dark_dae/link7_maste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; visual mesh filename=package://aloha_new_description/meshes/dark_dae/link7_maste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
- link bl_link8: geometry collision mesh filename=package://aloha_new_description/meshes/dark_dae/link8_maste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; visual mesh filename=package://aloha_new_description/meshes/dark_dae/link8_maste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
- link br_base_link: geometry collision mesh filename=package://aloha_new_description/meshes/dark_dae/base_link.d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; visual mesh filename=package://aloha_new_description/meshes/dark_dae/base_link.d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
- link br_link5: geometry collision mesh filename=package://aloha_new_description/meshes/dark_dae/link5.dae; visual mesh filename=package://aloha_new_description/meshes/dark_dae/link5.dae
- link br_link6: geometry collision mesh filename=package://aloha_new_description/meshes/dark_dae/link6_.dae; visual mesh filename=package://aloha_new_description/meshes/dark_dae/link6_.dae
- link br_link7: geometry collision mesh filename=package://aloha_new_description/meshes/dark_dae/link7_maste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; visual mesh filename=package://aloha_new_description/meshes/dark_dae/link7_maste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
- link br_link8: geometry collision mesh filename=package://aloha_new_description/meshes/dark_dae/link8_maste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; visual mesh filename=package://aloha_new_description/meshes/dark_dae/link8_maste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
- link fl_base_link: geometry collision mesh filename=package://aloha_new_description/meshes/dark_dae/base_link.d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; visual mesh filename=package://aloha_new_description/meshes/dark_dae/base_link.d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
- link fl_link5: geometry collision mesh filename=package://aloha_new_description/meshes/dark_dae/link5.dae; visual mesh filename=package://aloha_new_description/meshes/dark_dae/link5.dae
- link fr_base_link: geometry collision mesh filename=package://aloha_new_description/meshes/dark_dae/base_link.d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; visual mesh filename=package://aloha_new_description/meshes/dark_dae/base_link.d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
- link fr_link5: geometry collision mesh filename=package://aloha_new_description/meshes/dark_dae/link5.dae; visual mesh filename=package://aloha_new_description/meshes/dark_dae/link5.dae

File: aloha_new_description/urdf/aloha_tracer2_four_d435_dark.urdf (robot description, URDF)
Before this commit: robot aloha_description, 60 links, 59 joints
Links:
- link bl_base_link: geometry collision mesh filename=package://aloha_new_description/meshes/dark_dae/base_link.d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; visual mesh filename=package://aloha_new_description/meshes/dark_dae/base_link.d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
- link bl_link5: geometry collision mesh filename=package://aloha_new_description/meshes/dark_dae/link5.dae; visual mesh filename=package://aloha_new_description/meshes/dark_dae/link5.dae
- link bl_link6: geometry collision mesh filename=package://aloha_new_description/meshes/dark_dae/link6_.dae; visual mesh filename=package://aloha_new_description/meshes/dark_dae/link6_.dae
- link bl_link7: geometry collision mesh filename=package://aloha_new_description/meshes/dark_dae/link7_maste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; visual mesh filename=package://aloha_new_description/meshes/dark_dae/link7_maste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
- link bl_link8: geometry collision mesh filename=package://aloha_new_description/meshes/dark_dae/link8_maste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; visual mesh filename=package://aloha_new_description/meshes/dark_dae/link8_maste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
- link br_base_link: geometry collision mesh filename=package://aloha_new_description/meshes/dark_dae/base_link.d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; visual mesh filename=package://aloha_new_description/meshes/dark_dae/base_link.d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
- link br_link5: geometry collision mesh filename=package://aloha_new_description/meshes/dark_dae/link5.dae; visual mesh filename=package://aloha_new_description/meshes/dark_dae/link5.dae
- link br_link6: geometry collision mesh filename=package://aloha_new_description/meshes/dark_dae/link6_.dae; visual mesh filename=package://aloha_new_description/meshes/dark_dae/link6_.dae
- link br_link7: geometry collision mesh filename=package://aloha_new_description/meshes/dark_dae/link7_maste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; visual mesh filename=package://aloha_new_description/meshes/dark_dae/link7_maste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
- link br_link8: geometry collision mesh filename=package://aloha_new_description/meshes/dark_dae/link8_maste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; visual mesh filename=package://aloha_new_description/meshes/dark_dae/link8_maste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
- link fl_base_link: geometry collision mesh filename=package://aloha_new_description/meshes/dark_dae/base_link.d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; visual mesh filename=package://aloha_new_description/meshes/dark_dae/base_link.d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
- link fl_link5: geometry collision mesh filename=package://aloha_new_description/meshes/dark_dae/link5.dae; visual mesh filename=package://aloha_new_description/meshes/dark_dae/link5.dae
- link fr_base_link: geometry collision mesh filename=package://aloha_new_description/meshes/dark_dae/base_link.d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; visual mesh filename=package://aloha_new_description/meshes/dark_dae/base_link.d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
- link fr_link5: geometry collision mesh filename=package://aloha_new_description/meshes/dark_dae/link5.dae; visual mesh filename=package://aloha_new_description/meshes/dark_dae/link5.dae
- link mid_camera_stand_Link: geometry collision mesh filename=package://aloha_new_description/meshes/dark_dae/mid_double_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; visual mesh filename=package://aloha_new_description/meshes/dark_dae/mid_double_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
