Commit message: add piper camera

File: piper_description/urdf/piper_description_v100.urdf (robot description, URDF)
Before this commit: robot piper_camera, 9 links, 8 joints
Links:
- link arm_base: geometry collision mesh filename=package://piper_description/meshes/dae/base_link.dae; visual mesh filename=package://piper_description/meshes/dae/base_link.dae
- link link1: geometry collision mesh filename=package://piper_description/meshes/dae/link1.dae; visual mesh filename=package://piper_description/meshes/dae/link1.dae
- link link2: geometry collision mesh filename=package://piper_description/meshes/dae/link2.dae; visual mesh filename=package://piper_description/meshes/dae/link2.dae
- link link3: geometry collision mesh filename=package://piper_description/meshes/dae/link3.dae; visual mesh filename=package://piper_description/meshes/dae/link3.dae
- link link4: geometry collision mesh filename=package://piper_description/meshes/dae/link4.dae; visual mesh filename=package://piper_description/meshes/dae/link4.dae
- link link5: geometry collision mesh filename=package://piper_description/meshes/dae/link5.dae; visual mesh filename=package://piper_description/meshes/dae/link5.dae
- link link7: geometry collision mesh filename=package://piper_description/meshes/dae/link7.dae; visual mesh filename=package://piper_description/meshes/dae/link7.dae
- link link8: geometry collision mesh filename=package://piper_description/meshes/dae/link8.dae; visual mesh filename=package://piper_description/meshes/dae/link8.dae

File: piper_description/urdf/piper_description_v100_camera.urdf (robot description, URDF)
Before this commit: robot piper_camera, 0 links, 0 joints
Links:
- added link arm_base, mass 0.162548567403693; collision mesh filename=package://piper_description/meshes/dae/base_link.dae; visual mesh filename=package://piper_description/meshes/dae/base_link.dae
- added link link1, mass 0.0978679932242825; collision mesh filename=package://piper_description/meshes/dae/link1.dae; visual mesh filename=package://piper_description/meshes/dae/link1.dae
- added link link2, mass 0.290888938633388; collision mesh filename=package://piper_description/meshes/dae/link2.dae; visual mesh filename=package://piper_description/meshes/dae/link2.dae
- added link link3, mass 0.290847697793211; collision mesh filename=package://piper_description/meshes/dae/link3.dae; visual mesh filename=package://piper_description/meshes/dae/link3.dae
- added link link4, mass 0.127087348341362; collision mesh filename=package://piper_description/meshes/dae/link4.dae; visual mesh filename=package://piper_description/meshes/dae/link4.dae
- added link link5, mass 0.144711242639457; collision mesh filename=package://piper_description/meshes/dae/link5.dae; visual mesh filename=package://piper_description/meshes/dae/link5.dae
- added link link6, mass 0.195187143240719; collision mesh filename=package://piper_description/meshes/dae/camera_v3.dae; visual mesh filename=package://piper_description/meshes/dae/camera_v3.dae
- added link link7, mass 0.02648229234527; collision mesh filename=package://piper_description/meshes/dae/link7.dae; visual mesh filename=package://piper_description/meshes/dae/link7.dae
- added link link8, mass 0.0264822021416248; collision mesh filename=package://piper_description/meshes/dae/link8.dae; visual mesh filename=package://piper_description/meshes/dae/link8.dae
Joints:
- added joint joint1: type revolute, parent arm_base, child link1, origin xyz=0 0 0.123 rpy=0 0 -1.5708, axis 0 0 1, limit lower=-2.618 upper=2.618 effort=100 velocity=3
- added joint joint2: type revolute, parent link1, child link2, origin xyz=0 0 0 rpy=1.5708 -0.034907 -1.5708, axis 0 0 1, limit lower=0 upper=3.14 effort=100 velocity=3
- added joint joint3: type revolute, parent link2, child link3, origin xyz=0.28358 0.028726 0 rpy=0 0 0.06604341, axis 0 0 1, limit lower=-2.697 upper=0 effort=100 velocity=3
- added joint joint4: type revolute, parent link3, child link4, origin xyz=-0.24221 0.068514 0 rpy=-1.5708 0 1.3826, axis 0 0 1, limit lower=-1.832 upper=1.832 effort=100 velocity=3
- added joint joint5: type revolute, parent link4, child link5, origin xyz=0 0 0 rpy=1.5708 0 0, axis 0 0 1, limit lower=-1.22 upper=1.22 effort=100 velocity=3
- added joint joint6: type revolute, parent link5, child link6, origin xyz=0 0.091 0.0014165 rpy=-1.5708 -1.5708 0, axis 0 0 1, limit lower=-3.14 upper=3.14 effort=100 velocity=3
- added joint joint7: type prismatic, parent link6, child link7, origin xyz=0 0 0.13503 rpy=1.5708 0 1.5708, axis 0 0 -1, limit lower=0 upper=0.05 effort=10 velocity=1
- added joint joint8: type prismatic, parent link6, child link8, origin xyz=0 0 0.13503 rpy=-1.5708 0 1.5708, axis 0 0 1, limit lower=-0.05 upper=0 effort=10 velocity=1

File: piper_description/urdf/piper_description_with_camera_right.xacro (robot description, xacro)
@@ -19,5 +19,5 @@
         <origin xyz="0 0 0" rpy="0 0 0" />
         <geometry>
-            <mesh filename="package://aloha_new_description/meshes/base_link.dae" />
+            <mesh filename="package://piper_description/meshes/dae/base_link.dae" />
         </geometry>
         <material name="">
@@ -28,5 +28,5 @@
             <origin xyz="0 0 0" rpy="0 0 0" />
             <geometry>
-                <mesh filename="package://aloha_new_description/meshes/base_link.STL" />
+                <mesh filename="package://piper_description/meshes/dae/base_link.dae" />
             </geometry>
         </collision>
@@ -49,5 +49,5 @@
         <origin xyz="0 0 0" rpy="0 0 0" />
         <geometry>
-            <mesh filename="package://aloha_new_description/meshes/link1.dae" />
+            <mesh filename="package://piper_description/meshes/dae/link1.dae" />
         </geometry>
         <material name="">
@@ -58,5 +58,5 @@
             <origin xyz="0 0 0" rpy="0 0 0" />
             <geometry>
-                <mesh filename="package://aloha_new_description/meshes/link1.STL" />
+                <mesh filename="package://piper_description/meshes/dae/link1.dae" />
             </geometry>
         </collision>
@@ -86,5 +86,5 @@
         <origin xyz="0 0 0" rpy="0 0 0" />
         <geometry>
-            <mesh filename="package://aloha_new_description/meshes/link2.dae" />
+            <mesh filename="package://piper_description/meshes/dae/link2.dae" />
         </geometry>
         <material name="">
@@ -95,5 +95,5 @@
             <origin xyz="0 0 0" rpy="0 0 0" />
             <geometry>
-                <mesh filename="package://aloha_new_description/meshes/link2.STL" />
+                <mesh filename="package://piper_description/meshes/dae/link2.dae" />
             </geometry>
         </collision>
@@ -123,14 +123,14 @@
         <origin xyz="0 0 0" rpy="0 0 0" />
         <geometry>
-            <mesh filename="package://aloha_new_description/meshes/link3.dae" />
-        </geometry>
-        <material name="">
-            <color rgba="0.792156862745098 0.819607843137255 0.933333333333333 1" />
-        </material>
-        </visual>
-        <collision>
-        <origin xyz="0 0 0" rpy="0 0 0" />
-        <geometry>
-            <mesh filename="package://aloha_new_description/meshes/link3.STL" />
+            <mesh filename="package://piper_description/meshes/dae/link3.dae" />
+        </geometry>
+        <material name="">
+            <color rgba="0.792156862745098 0.819607843137255 0.933333333333333 1" />
+        </material>
+        </visual>
+        <collision>
+        <origin xyz="0 0 0" rpy="0 0 0" />
+        <geometry>
+            <mesh filename="package://piper_description/meshes/dae/link3.dae" />
         </geometry>
         </collision>
@@ -160,14 +160,14 @@
         <origin xyz="0 0 0" rpy="0 0 0" />
         <geometry>
-            <mesh filename="package://aloha_new_description/meshes/link4.dae" />
-        </geometry>
-        <material name="">
-            <color rgba="0.792156862745098 0.819607843137255 0.933333333333333 1" />
-        </material>
-        </visual>
-        <collision>
-        <origin xyz="0 0 0" rpy="0 0 0" />
-        <geometry>
-            <mesh filename="package://aloha_new_description/meshes/link4.STL" />
+            <mesh filename="package://piper_description/meshes/dae/link4.dae" />
+        </geometry>
+        <material name="">
+            <color rgba="0.792156862745098 0.819607843137255 0.933333333333333 1" />
+        </material>
+        </visual>
+        <collision>
+        <origin xyz="0 0 0" rpy="0 0 0" />
+        <geometry>
+            <mesh filename="package://piper_description/meshes/dae/link4.dae" />
         </geometry>
         </collision>
@@ -197,14 +197,14 @@
         <origin xyz="0 0 0" rpy="0 0 0" />
         <geometry>
-            <mesh filename="package://aloha_new_description/meshes/link5.dae" />
-        </geometry>
-        <material name="">
-            <color rgba="0.792156862745098 0.819607843137255 0.933333333333333 1" />
-        </material>
-        </visual>
-        <collision>
-        <origin xyz="0 0 0" rpy="0 0 0" />
-        <geometry>
-            <mesh filename="package://aloha_new_description/meshes/link5.STL" />
+            <mesh filename="package://piper_description/meshes/dae/link5.dae" />
+        </geometry>
+        <material name="">
+            <color rgba="0.792156862745098 0.819607843137255 0.933333333333333 1" />
+        </material>
+        </visual>
+        <collision>
+        <origin xyz="0 0 0" rpy="0 0 0" />
+        <geometry>
+            <mesh filename="package://piper_description/meshes/dae/link5.dae" />
         </geometry>
         </collision>
@@ -232,17 +232,16 @@
         </inertial>
         <visual>
-        <origin xyz="-0.002 -0.0078 0.06" rpy="-1.57 0 0" />
-        <geometry>
-            <mesh filename="package://aloha_new_description/meshes/piper_slave_meshes/gripper_base_100_v2.dae"/>
-        </geometry>
-        <material name="">
-            <color rgba="0.792156862745098 0.819607843137255 0.933333333333333 1" />
-        </material>
-        </visual>
-        <collision>
-        <origin xyz="0 0 0" rpy="0 0 0" />
-        <origin xyz="-0.002 -0.0078 0.06" rpy="-1.57 0 0" />
-        <geometry>
-            <mesh filename="package://aloha_new_description/meshes/piper_slave_meshes/gripper_base_100_v2.dae"/>
+        <origin xyz="-0.002 -0.008 0" rpy="-1.57 0 0" />
+        <geometry>
+            <mesh filename="package://piper_description/meshes/dae/camera_v3.dae"/>
+        </geometry>
+        <material name="">
+            <color rgba="0.792156862745098 0.819607843137255 0.933333333333333 1" />
+        </material>
+        </visual>
+        <collision>
+        <origin xyz="-0.002 -0.008 0" rpy="-1.57 0 0" />
+        <geometry>
+            <mesh filename="package://piper_description/meshes/dae/camera_v3.dae"/>
         </geometry>
         </collision>
@@ -272,14 +271,14 @@
         <origin xyz="0 0 0" rpy="0 0 0" />
         <geometry>
-            <mesh filename="package://aloha_new_description/meshes/piper_slave_meshes/link7.dae" />
-        </geometry>
-        <material name="">
-            <color rgba="0.792156862745098 0.819607843137255 0.933333333333333 1" />
-        </material>
-        </visual>
-        <collision>
-        <origin xyz="0 0 0" rpy="0 0 0" />
-        <geometry>
-            <mesh filename="package://aloha_new_description/meshes/piper_slave_meshes/link7.STL" />
+            <mesh filename="package://piper_description/meshes/dae/link7.dae" />
+        </geometry>
+        <material name="">
+            <color rgba="0.792156862745098 0.819607843137255 0.933333333333333 1" />
+        </material>
+        </visual>
+        <collision>
+        <origin xyz="0 0 0" rpy="0 0 0" />
+        <geometry>
+            <mesh filename="package://piper_description/meshes/dae/link7.dae" />
         </geometry>
         </collision>
@@ -290,5 +289,5 @@
         <child link="${namespace}/link7" />
         <axis xyz="0 0 -1" />
-        <limit lower="0" upper="0.04" effort="10" velocity="1" />
+        <limit lower="0" upper="0.05" effort="10" velocity="1" />
     </joint>
     <link name="${namespace}/link8">
@@ -309,14 +308,14 @@
         <origin xyz="0 0 0" rpy="0 0 0" />
         <geometry>
-            <mesh filename="package://aloha_new_description/meshes/piper_slave_meshes/link8.dae" />
-        </geometry>
-        <material name="">
-            <color rgba="0.792156862745098 0.819607843137255 0.933333333333333 1" />
-        </material>
-        </visual>
-        <collision>
-        <origin xyz="0 0 0" rpy="0 0 0" />
-        <geometry>
-            <mesh filename="package://aloha_new_description/meshes/piper_slave_meshes/link8.STL" />
+            <mesh filename="package://piper_description/meshes/dae/link8.dae" />
+        </geometry>
+        <material name="">
+            <color rgba="0.792156862745098 0.819607843137255 0.933333333333333 1" />
+        </material>
+        </visual>
+        <collision>
+        <origin xyz="0 0 0" rpy="0 0 0" />
+        <geometry>
+            <mesh filename="package://piper_description/meshes/dae/link8.dae" />
         </geometry>
         </collision>
@@ -327,5 +326,5 @@
         <child link="${namespace}/link8" />
         <axis xyz="0 0 1" />
-        <limit lower="-0.04" upper="0" effort="10" velocity="1" />
+        <limit lower="-0.05" upper="0" effort="10" velocity="1" />
     </joint>
 </xacro:macro>

File: split_aloha_mid_360/urdf/split_aloha_mid_360_with_piper.xacro (robot description, xacro)
@@ -3,6 +3,6 @@
 <xacro:include filename="$(find split_aloha_mid_360)/urdf/split_aloha_mid_360.xacro"/>
 <!-- <xacro:include filename="$(find piper_description)/urdf/piper_description_left.xacro"/> -->
-<xacro:include filename="$(find piper_description)/urdf/piper_description_left.xacro"/>
-<xacro:include filename="$(find piper_description)/urdf/piper_description_right.xacro"/>
+<xacro:include filename="$(find piper_description)/urdf/piper_description_with_camera_left.xacro"/>
+<xacro:include filename="$(find piper_description)/urdf/piper_description_with_camera_right.xacro"/>
 <!-- <xacro:include filename="$(find piper_description)/urdf/piper_description_right.xacro"/> -->
 <xacro:left_arm namespace="left">
