Commit message: update collision model

File: piper_description/urdf/piper_description_v100.urdf (robot description, URDF)
Before this commit: robot piper_camera, 9 links, 8 joints
Links:
- link arm_base: geometry collision mesh filename=package://piper_description/meshes/base_link.STL; visual mesh filename=package://piper_description/meshes/dae/base_link.dae
- link link1: geometry collision mesh filename=package://piper_description/meshes/link1.STL; visual mesh filename=package://piper_description/meshes/dae/link1.dae
- link link2: geometry collision mesh filename=package://piper_description/meshes/link2.STL; visual mesh filename=package://piper_description/meshes/dae/link2.dae
- link link3: geometry collision mesh filename=package://piper_description/meshes/link3.STL; visual mesh filename=package://piper_description/meshes/dae/link3.dae
- link link4: geometry collision mesh filename=package://piper_description/meshes/link4.STL; visual mesh filename=package://piper_description/meshes/dae/link4.dae
- link link5: geometry collision mesh filename=package://piper_description/meshes/link5.STL; visual mesh filename=package://piper_description/meshes/dae/link5.dae
- link link7: geometry collision mesh filename=package://piper_description/meshes/link7.STL; visual mesh filename=package://piper_description/meshes/dae/link7.dae
- link link8: geometry collision mesh filename=package://piper_description/meshes/link8.STL; visual mesh filename=package://piper_description/meshes/dae/link8.dae

File: piper_description/urdf/piper_description_v100_camera.urdf (robot description, URDF)
Before this commit: robot piper_camera, 9 links, 8 joints
Links:
- link arm_base: geometry collision mesh filename=package://piper_description/meshes/base_link.STL; visual mesh filename=package://piper_description/meshes/dae/base_link.dae
- link link1: geometry collision mesh filename=package://piper_description/meshes/link1.STL; visual mesh filename=package://piper_description/meshes/dae/link1.dae
- link link2: geometry collision mesh filename=package://piper_description/meshes/link2.STL; visual mesh filename=package://piper_description/meshes/dae/link2.dae
- link link3: geometry collision mesh filename=package://piper_description/meshes/link3.STL; visual mesh filename=package://piper_description/meshes/dae/link3.dae
- link link4: geometry collision mesh filename=package://piper_description/meshes/link4.STL; visual mesh filename=package://piper_description/meshes/dae/link4.dae
- link link5: geometry collision mesh filename=package://piper_description/meshes/link5.STL; visual mesh filename=package://piper_description/meshes/dae/link5.dae
- link link7: geometry collision mesh filename=package://piper_description/meshes/link7.STL; visual mesh filename=package://piper_description/meshes/dae/link7.dae
- link link8: geometry collision mesh filename=package://piper_description/meshes/link8.STL; visual mesh filename=package://piper_description/meshes/dae/link8.dae

File: piper_description/urdf/piper_description_with_camera_left.xacro (robot description, xacro)
@@ -28,5 +28,5 @@
             <origin xyz="0 0 0" rpy="0 0 0" />
             <geometry>
-                <mesh filename="package://piper_description/meshes/dae/base_link.dae" />
+                <mesh filename="package://piper_description/meshes/base_link.STL" />
             </geometry>
         </collision>
@@ -56,7 +56,7 @@
         </visual>
         <collision>
-            <origin xyz="0 0 0" rpy="0 0 0" />
+            <origin xyz="0 0 0" rpy="0 0 1.5708" />
             <geometry>
-                <mesh filename="package://piper_description/meshes/dae/link1.dae" />
+                <mesh filename="package://piper_description/meshes/link1.STL" />
             </geometry>
         </collision>
@@ -93,7 +93,7 @@
         </visual>
         <collision>
-            <origin xyz="0 0 0" rpy="0 0 0" />
+            <origin xyz="0 0 0" rpy="0 0 0.1" />
             <geometry>
-                <mesh filename="package://piper_description/meshes/dae/link2.dae" />
+                <mesh filename="package://piper_description/meshes/link2.STL" />
             </geometry>
         </collision>
@@ -130,7 +130,7 @@
         </visual>
         <collision>
-        <origin xyz="0 0 0" rpy="0 0 0" />
-        <geometry>
-            <mesh filename="package://piper_description/meshes/dae/link3.dae" />
+        <origin xyz="0 0 0" rpy="0 0 -1.75" />
+        <geometry>
+            <mesh filename="package://piper_description/meshes/link3.STL" />
         </geometry>
         </collision>
@@ -169,5 +169,5 @@
         <origin xyz="0 0 0" rpy="0 0 0" />
         <geometry>
-            <mesh filename="package://piper_description/meshes/dae/link4.dae" />
+            <mesh filename="package://piper_description/meshes/link4.STL" />
         </geometry>
         </collision>
@@ -204,7 +204,7 @@
         </visual>
         <collision>
-        <origin xyz="0 0 0" rpy="0 0 0" />
-        <geometry>
-            <mesh filename="package://piper_description/meshes/dae/link5.dae" />
+        <origin xyz="0 0 0" rpy="0 0 -3.14" />
+        <geometry>
+            <mesh filename="package://piper_description/meshes/link5.STL" />
         </geometry>
         </collision>
@@ -278,7 +278,7 @@
         </visual>
         <collision>
-        <origin xyz="0 0 0" rpy="0 0 0" />
-        <geometry>
-            <mesh filename="package://piper_description/meshes/dae/link7.dae" />
+        <origin xyz="-0.001 0 0.0003" rpy="0 3.14 0" />
+        <geometry>
+            <mesh filename="package://piper_description/meshes/link7.STL" />
         </geometry>
         </collision>
@@ -315,7 +315,7 @@
         </visual>
         <collision>
-        <origin xyz="0 0 0" rpy="0 0 0" />
-        <geometry>
-            <mesh filename="package://piper_description/meshes/dae/link8.dae" />
+        <origin xyz="-0.001 0 0.0003" rpy="3.14 0 0" />
+        <geometry>
+            <mesh filename="package://piper_description/meshes/link8.STL" />
         </geometry>
         </collision>

File: piper_description/urdf/piper_description_with_camera_right.xacro (robot description, xacro)
@@ -28,5 +28,5 @@
             <origin xyz="0 0 0" rpy="0 0 0" />
             <geometry>
-                <mesh filename="package://piper_description/meshes/dae/base_link.dae" />
+                <mesh filename="package://piper_description/meshes/base_link.STL" />
             </geometry>
         </collision>
@@ -56,7 +56,7 @@
         </visual>
         <collision>
-            <origin xyz="0 0 0" rpy="0 0 0" />
+            <origin xyz="0 0 0" rpy="0 0 1.5708" />
             <geometry>
-                <mesh filename="package://piper_description/meshes/dae/link1.dae" />
+                <mesh filename="package://piper_description/meshes/link1.STL" />
             </geometry>
         </collision>
@@ -93,7 +93,7 @@
         </visual>
         <collision>
-            <origin xyz="0 0 0" rpy="0 0 0" />
+            <origin xyz="0 0 0" rpy="0 0 0.1" />
             <geometry>
-                <mesh filename="package://piper_description/meshes/dae/link2.dae" />
+                <mesh filename="package://piper_description/meshes/link2.STL" />
             </geometry>
         </collision>
@@ -130,7 +130,7 @@
         </visual>
         <collision>
-        <origin xyz="0 0 0" rpy="0 0 0" />
-        <geometry>
-            <mesh filename="package://piper_description/meshes/dae/link3.dae" />
+        <origin xyz="0 0 0" rpy="0 0 -1.75" />
+        <geometry>
+            <mesh filename="package://piper_description/meshes/link3.STL" />
         </geometry>
         </collision>
@@ -169,5 +169,5 @@
         <origin xyz="0 0 0" rpy="0 0 0" />
         <geometry>
-            <mesh filename="package://piper_description/meshes/dae/link4.dae" />
+            <mesh filename="package://piper_description/meshes/link4.STL" />
         </geometry>
         </collision>
@@ -204,7 +204,7 @@
         </visual>
         <collision>
-        <origin xyz="0 0 0" rpy="0 0 0" />
-        <geometry>
-            <mesh filename="package://piper_description/meshes/dae/link5.dae" />
+        <origin xyz="0 0 0" rpy="0 0 -3.14" />
+        <geometry>
+            <mesh filename="package://piper_description/meshes/link5.STL" />
         </geometry>
         </collision>
@@ -278,7 +278,7 @@
         </visual>
         <collision>
-        <origin xyz="0 0 0" rpy="0 0 0" />
-        <geometry>
-            <mesh filename="package://piper_description/meshes/dae/link7.dae" />
+        <origin xyz="-0.001 0 0.0003" rpy="0 3.14 0" />
+        <geometry>
+            <mesh filename="package://piper_description/meshes/link7.STL" />
         </geometry>
         </collision>
@@ -315,7 +315,7 @@
         </visual>
         <collision>
-        <origin xyz="0 0 0" rpy="0 0 0" />
-        <geometry>
-            <mesh filename="package://piper_description/meshes/dae/link8.dae" />
+        <origin xyz="-0.001 0 0.0003" rpy="3.14 0 0" />
+        <geometry>
+            <mesh filename="package://piper_description/meshes/link8.STL" />
         </geometry>
         </collision>

File: split_aloha_mid_360/urdf/ranger_mini.xacro (robot description, xacro)
@@ -183,5 +183,5 @@
             </visual>
             <collision>
-                <origin xyz="0 0 0" rpy="1.57 0 0" />
+                <origin xyz="0 0 -0.005" rpy="1.57 0 0" />
                 <geometry>
                     <cylinder length="0.08" radius="0.09" />
@@ -267,5 +267,5 @@
             </visual>
             <collision>
-                <origin xyz="0.005 0.005 -0.005" rpy="1.57 0 0" />
+                <origin xyz="0.00 0.00 -0.005" rpy="1.57 0 0" />
                 <geometry>
                     <cylinder length="0.08" radius="0.09" />
@@ -325,5 +325,5 @@
             </visual>
             <collision>
-                <origin xyz="-0.015 0.02 -0.005" rpy="1.57 0 0" />
+                <origin xyz="0.00 0 -0.005" rpy="1.57 0 0" />
                 <geometry>
                     <cylinder length="0.08" radius="0.09" />
