Commit message: 修复URDF

File: piper_description/urdf/piper_description_left.xacro (robot description, xacro)
@@ -28,5 +28,5 @@
             <origin xyz="0 0 0" rpy="0 0 0" />
             <geometry>
-                <mesh filename="package://piper_description/meshes/base_link.STL" />
+            <mesh filename="package://piper_description/meshes/dae/base_link.dae" />
             </geometry>
         </collision>

File: piper_description/urdf/piper_description_right.xacro (robot description, xacro)
@@ -28,5 +28,5 @@
             <origin xyz="0 0 0" rpy="0 0 0" />
             <geometry>
-                <mesh filename="package://piper_description/meshes/base_link.STL" />
+            <mesh filename="package://piper_description/meshes/dae/base_link.dae" />
             </geometry>
         </collision>

File: piper_description/urdf/piper_description_with_camera_left.xacro (robot description, xacro)
@@ -28,5 +28,5 @@
             <origin xyz="0 0 0" rpy="0 0 0" />
             <geometry>
-                <mesh filename="package://piper_description/meshes/base_link.STL" />
+            <mesh filename="package://piper_description/meshes/dae/base_link.dae" />
             </geometry>
         </collision>

File: piper_description/urdf/piper_description_with_camera_right.xacro (robot description, xacro)
@@ -28,5 +28,5 @@
             <origin xyz="0 0 0" rpy="0 0 0" />
             <geometry>
-                <mesh filename="package://piper_description/meshes/base_link.STL" />
+            <mesh filename="package://piper_description/meshes/dae/base_link.dae" />
             </geometry>
         </collision>

File: split_aloha_mid_360/urdf/split_aloha_mid_360_with_piper.urdf (robot description, URDF)
Before this commit: robot split_aloha_mid_360_with_piper, 32 links, 31 joints
Links:
- link left/arm_base: geometry collision mesh filename=package://piper_description/meshes/dae/base_link.dae; visual mesh filename=package://piper_description/meshes/dae/base_link.dae
- link left/link6: geometry collision mesh filename=package://piper_description/meshes/dae/camera_v3.dae; visual mesh filename=package://piper_description/meshes/dae/camera_v3.dae
- link right/arm_base: geometry collision mesh filename=package://piper_description/meshes/dae/base_link.dae; visual mesh filename=package://piper_description/meshes/dae/base_link.dae
- link right/link6: geometry collision mesh filename=package://piper_description/meshes/dae/camera_v3.dae; visual mesh filename=package://piper_description/meshes/dae/camera_v3.dae

File: split_aloha_mid_360/urdf/split_aloha_rslidar_with_piper.urdf (robot description, URDF)
Before this commit: robot split_aloha_rslidar_with_piper, 32 links, 31 joints
Links:
- link left/arm_base: geometry collision mesh filename=package://piper_description/meshes/dae/base_link.dae; visual mesh filename=package://piper_description/meshes/dae/base_link.dae
- link right/arm_base: geometry collision mesh filename=package://piper_description/meshes/dae/base_link.dae; visual mesh filename=package://piper_description/meshes/dae/base_link.dae
