Commit message: 更新升降柱限位

File: split_aloha_mid_360/urdf/split_aloha_mid_360.xacro (robot description, xacro)
@@ -205,5 +205,5 @@
     type="prismatic">
     <origin
-      xyz="0.22448 0 1.1147"
+      xyz="0.22448 0 0.3147"
       rpy="0 0 0" />
     <parent
@@ -213,5 +213,5 @@
     <axis
       xyz="0 0 1" />
-    <limit lower="-0.6" upper="0.0" effort="100" velocity="10.0"/>
+    <limit lower="0.0" upper="0.8" effort="100" velocity="10.0"/>
   </joint>
   <link
